Commit message: Restored the progress and reconneted the right email

File: URDF/plotter.urdf (robot description, URDF)
Before this commit: robot cartesian_plotter, 2 links, 1 joints
Links:
- added link base_link, mass 1.0; visual mesh filename=file:///home/vaibhav/programming_projects/Robotics/Cartesia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 scale=.05 .05 .05
- link X_Rail: geometry visual mesh filename=file:///home/vaibhav/programming_projects/Robotics/Cartesia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 scale=.05 .05 .05
- link Y_rail: geometry visual mesh filename=file:///home/vaibhav/programming_projects/Robotics/Cartesia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 scale=.05 .05 .05
Joints:
- added joint base_to_x: type fixed, parent base_link, child X_Rail, origin xyz=0 0 0 rpy=0 0 0
- joint x_to_y: axis (none) -> 1 0 0; limit (none) -> lower=0 upper=5000 effort=10 velocity=1; origin xyz=0 0 .10 rpy=0 0 0 -> xyz=0 0 0 rpy=0 0 0; type fixed -> prismatic

Commit message: Added joint controller plugin and damping in joint

File: URDF/plotter.urdf (robot description, URDF)
Before this commit: robot cartesian_plotter, 3 links, 2 joints
Links:
- added link world
Joints:
- added joint world_to_base: type fixed, parent world, child base_link, origin xyz=0 0 0 rpy=0 0 0
- joint x_to_y: limit lower=0 upper=5000 effort=10 velocity=1 -> lower=0 upper=0.5 effort=100 velocity=1

Commit message: Added paper and made some changes to PID loop

File: URDF/plotter.urdf (robot description, URDF)
Before this commit: robot cartesian_plotter, 6 links, 5 joints
Links:
- added link paper, mass 0.03; collision box size=0.297 0.210 0.001; visual box size=0.297 0.210 0.001
Joints:
- added joint pen and base: type fixed, parent base_link, child paper, origin xyz=0 0 0.05 rpy=0 0 0
